File: PCB/DCI_TP_Final_GG/DCI_TP_Final_GG.kicad_pcb (KiCad board)
At the start: 2 copper layers, 42 x 90 mm, 70 parts, among them J201 DRIVER A OUT, J301 DRIVER B OUT, J401 IN - Driver A, J402 IN - Driver B, J403 Vin, J404 Vout, U201 A3967, U301 A3967, U401 LM317

Commit message: Cambio Versión en PCB
Other:
- board text added: "V1.0 - 10/19"
- board text removed: "V1019"
Changed lines of the file:
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@@
   (general
     (thickness 1.6)
-    (drawings 11)
+    (drawings 10)
     (tracks 568)
     (zones 0)
@@
   )
   (layers
-    (0 F.Cu signal hide)
-    (31 B.Cu signal hide)
-    (32 B.Adhes user hide)
-    (33 F.Adhes user hide)
-    (34 B.Paste user hide)
-    (35 F.Paste user hide)
-    (36 B.SilkS user hide)
+    (0 F.Cu signal)
+    (31 B.Cu signal)
+    (32 B.Adhes user)
+    (33 F.Adhes user)
+    (34 B.Paste user)
+    (35 F.Paste user)
+    (36 B.SilkS user)
     (37 F.SilkS user)
-    (38 B.Mask user hide)
-    (39 F.Mask user hide)
-    (40 Dwgs.User user hide)
-    (41 Cmts.User user hide)
-    (42 Eco1.User user hide)
-    (43 Eco2.User user hide)
-    (44 Edge.Cuts user hide)
-    (45 Margin user hide)
-    (46 B.CrtYd user hide)
-    (47 F.CrtYd user hide)
-    (48 B.Fab user hide)
-    (49 F.Fab user hide)
+    (38 B.Mask user)
+    (39 F.Mask user)
+    (40 Dwgs.User user)
+    (41 Cmts.User user)
+    (42 Eco1.User user)
+    (43 Eco2.User user)
+    (44 Edge.Cuts user)
+    (45 Margin user)
+    (46 B.CrtYd user)
+    (47 F.CrtYd user)
+    (48 B.Fab user)
+    (49 F.Fab user)
   )
   (setup
@@
     (descr "CP, Radial series, Radial, pin pitch=2.00mm, , diameter=5mm, Electrolytic Capacitor")
     (tags "CP Radial series Radial pin pitch 2.00mm  diameter 5mm Electrolytic Capacitor")
-    (fp_text reference C303 (at 1 -3.75) (layer F.SilkS)
-      (effects (font (size 1 1) (thickness 0.15)))
+    (fp_text reference C303 (at 0.5 -3.9) (layer F.SilkS)
+      (effects (font (size 0.7 0.7) (thickness 0.15)))
     )
     (fp_text value "47uF x 35V" (at 1 3.75) (layer F.Fab)
@@
     (tags "Potentiometer vertical Vishay TS53YJ")
     (attr smd)
-    (fp_text reference RV301 (at 2 -3.5 90) (layer F.SilkS)
-      (effects (font (size 0.75 0.75) (thickness 0.15)))
+    (fp_text reference RV301 (at 2.2 -3.3 90) (layer F.SilkS)
+      (effects (font (size 0.7 0.7) (thickness 0.15)))
     )
     (fp_text value 10k (at -1 3.5 90) (layer F.Fab)
@@
     (tags resistor)
     (attr smd)
-    (fp_text reference R310 (at 0.25 -1.65 90) (layer F.SilkS)
-      (effects (font (size 1 1) (thickness 0.15)))
+    (fp_text reference R310 (at 0.1 -1.6 90) (layer F.SilkS)
+      (effects (font (size 0.7 0.7) (thickness 0.15)))
     )
     (fp_text value 0.75 (at 0 1.65 90) (layer F.Fab)
@@
     (tags resistor)
     (attr smd)
-    (fp_text reference R303 (at -3.5625 0) (layer F.SilkS)
-      (effects (font (size 1 1) (thickness 0.15)))
+    (fp_text reference R303 (at -3.0625 0) (layer F.SilkS)
+      (effects (font (size 0.7 0.7) (thickness 0.15)))
     )
     (fp_text value 10K (at 0 1.65) (layer F.Fab)
@@
     )
   )
-  (gr_text "Grilla componentes: 5mm, 2,5mm,\n 1mm y 0.5mm(para ajuste fino en\nel control de clearance)\n\nGrilla pistas: 1mm, 0.5mm, 0.25mm \ny 0.1 (para ajuste fino)\n\nVias: 1.3mm ,1.5mm y 2mm (Limite Mayer=1.27)\n\nAgujeros: 0.8mm,0.9mm , 1mm , 1.3mm y 3mm\n(Limite Mayer = 0.7mm)\n\nPistas: 0.5mm, 0.75mm, 1mm, 1.5mm, 2mm\n(limite Mayer = 0.3mm)\n\nClearance > 0.3 mm  (Limite Mayer=0.3mm)\n\nPCB\nSustrato: FR4 - 1.6mm de espesor\nCobre: 1 Oz\nTerminación: HASL\n\n" (at 140 87.5) (layer Dwgs.User)
-    (effects (font (size 1 1) (thickness 0.15)) (justify left))
-  )
-  (gr_text V1019 (at 130 135) (layer B.Cu)
+  (gr_text "V1.0 - 10/19" (at 130 135) (layer B.Cu)
     (effects (font (size 1.5 1.5) (thickness 0.3)) (justify mirror))
   )
@@
     (arrow2b (pts (xy 106.5 44.5) (xy 107.626504 43.913579)))
   )
-  (gr_text "Grilla componentes: 5mm, 2,5mm,\n 1mm y 0.5mm(para ajuste fino en\nel control de clearance)\n\nGrilla pistas: 1mm, 0.5mm, 0.25mm \ny 0.1 (para ajuste fino)\n\nVias: 1.3mm ,1.5mm y 2mm (Limite Mayer=1.27)\n\nAgujeros: 0.8mm,0.9mm , 1mm , 1.3mm y 3mm\n(Limite Mayer = 0.7mm)\n\nPistas: 0.5mm, 0.75mm, 1mm, 1.5mm, 2mm\n(limite Mayer = 0.3mm)\n\nClearance > 0.3 mm  (Limite Mayer=0.3mm)\n\nPCB\nSustrato: FR4 - 1.6mm de espesor\nCobre: 1 Oz\nTerminación: HASL\n\n" (at 175.5 87) (layer Dwgs.User)
+  (gr_text "Grilla componentes: 5mm, 2,5mm,\n 1mm y 0.5mm(para ajuste fino en\nel control de clearance)\n\nGrilla pistas: 1mm, 0.5mm, 0.25mm \ny 0.1 (para ajuste fino)\n\nVias: 1.3mm ,1.5mm y 2mm (Limite Mayer=1.27)\n\nAgujeros: 0.8mm,0.9mm , 1mm , 1.3mm y 3mm\n(Limite Mayer = 0.7mm)\n\nPistas: 0.5mm, 0.75mm, 1mm, 1.5mm, 2mm\n(limite Mayer = 0.3mm)\n\nClearance > 0.3 mm  (Limite Mayer=0.3mm)\n\nPCB\nSustrato: FR4 - 1.6mm de espesor\nCobre: 1 Oz\nTerminación: HASL\n\n" (at 175.5 87) (layer Cmts.User)
     (effects (font (size 1 1) (thickness 0.15)) (justify left))
   )
@@
       )
     )
+  )
+  (zone (net 0) (net_name "") (layer B.Cu) (hatch edge 0.508)
+    (connect_pads (clearance 0.508))
+    (min_thickness 0.254)
+    (keepout (tracks allowed) (vias allowed) (copperpour not_allowed))
+    (fill (arc_segments 32) (thermal_gap 0.508) (thermal_bridge_width 0.508))
+    (polygon
+      (pts
+        (xy 109.5 107.5) (xy 109.5 130) (xy 112.5 130) (xy 112.5 107.5)
+      )
+    )
+  )
+  (zone (net 0) (net_name "") (layer B.Cu) (hatch edge 0.508)
+    (connect_pads (clearance 0.508))
+    (min_thickness 0.254)
+    (keepout (tracks allowed) (vias allowed) (copperpour not_allowed))
+    (fill (arc_segments 32) (thermal_gap 0.508) (thermal_bridge_width 0.508))
+    (polygon
+      (pts
+        (xy 109.5 63.5) (xy 109.5 86) (xy 112.5 86) (xy 112.5 63.5)
+      )
+    )
